File: indexspeakerdacdev/indexspeakerdac.kicad_pcb (KiCad board)
At the start: 2 copper layers, 11 x 29.2 mm, 41 parts, among them IC1 MAX98360AEFB+T, IC2 MAX98360AEFB+T, IC3 W25Q16JVUXIQ_TR, J1 Conn_01x04_Pin, J2 Conn_01x11_Pin, J3 Conn_01x01_Pin, J4 Conn_01x11_Pin, J5 Conn_01x01_Pin, J6 USB_C_Plug_USB2.0, U1 RP2040, U2 MIC5317-3.3xM5, Y1 Crystal_GND24

Commit message: Add files via upload
Parts:
- added R6: 5.1K, Resistor_SMD:R_0201_0603Metric, F.Cu at (140.4, 101.0)
- J6: value USB_C_Plug_USB2.0 -> USB_C_Receptacle_USB2.0
- moved R5 2.00 mm to (138.3, 100.8), turned to -90 degrees
Connections:
- J6 pad A8: (no net) -> unconnected-(J6-SBU1-PadA8)
- J6 pad B5: unconnected-(J6-VCONN-PadB5) -> Net-(J6-CC2)
- J6 pad B6: (no net) -> /D+
- J6 pad B7: (no net) -> /D-
- J6 pad B8: (no net) -> unconnected-(J6-SBU2-PadB8)
Routing:
- net VCC: track 50.4 -> 45.8 mm
- net Net-(J6-CC2): track 0.00 -> 3.56 mm
- net Net-(J6-CC1): track 1.97 -> 4.44 mm
- net /D+: track 5.41 -> 6.97 mm, vias 2 -> 0
- net /D-: track 5.88 -> 7.30 mm, vias 0 -> 2
- added copper zone on B.Cu, net VCC
Other:
- board text added: "BOOTSEL"
- board text removed: "BOOT"
